File: boomdsp.brd (EAGLE design)
At the start: 100 x 100 mm, 20 parts

Commit message: damn vias
Parts:
- removed C5, C7: 2.2uF 25V, rcl:C0805
- removed I2C: 1X2, headers(2mm):1X2
- removed U$2: 1X4, headers(2mm):1X4
- added C2, C9: (no value), rcl:C1206
- added H1, H2, H3, H4: MOUNT-HOLE3.2, holes:3,2
- added SV2: (no value), con-lstb:MA06-1
- moved R1 12.4 mm to (21.5, 17.7)
- moved R2 12.3 mm to (26.3, 17.8)
- moved I2S 12.2 mm to (26.4, 39.4)
- moved U$4 12.2 mm to (20.4, 39.4)
- moved C4 12.0 mm to (18.4, 31.9)
- moved C3 10.8 mm to (19.4, 35.4)
- moved C13 10.7 mm to (16.4, 12.4)
- moved C14 10.7 mm to (31.4, 12.4)
- moved OUTL 10.7 mm to (20.4, 8.90)
- moved OUTR 10.7 mm to (27.4, 8.90)
- moved POWER 10.7 mm to (11.4, 26.9)
- moved POWER1 10.7 mm to (11.4, 32.9)
- moved U$1 10.7 mm to (24.6, 28.7)
- moved C1 10.7 mm to (32.9, 19.9)
- moved C6 10.7 mm to (18.4, 26.9)
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Connections:
- net GND: now also C2.1; no longer C5.1
- net N$10: now also SV2.4; no longer U$2.3
- net N$11: now also SV2.6; no longer U$2.1
- net N$12: now also C9.1; no longer C7.1
- net N$19: now also SV2.1; no longer I2C.1
- net N$20: now also SV2.2; no longer I2C.2
- net N$5: now also C9.2; no longer C7.2
- net N$7: now also SV2.5; no longer U$2.2
- net N$8: now also SV2.3; no longer U$2.4
- net N$9: now also C2.2; no longer C5.2
Routing:
- net GND: track 4.34 -> 17.4 mm, vias 6 -> 0
- net N$11: track 7.60 -> 14.5 mm
- net N$7: track 3.83 -> 9.19 mm
- net N$8: track 4.97 -> 10.1 mm
- net N$20: track 6.09 -> 10.8 mm
- net N$19: track 6.53 -> 11.0 mm
- net N$10: track 7.16 -> 11.5 mm
- net VCC: track 39.2 -> 35.3 mm
- net N$21: track 6.10 -> 8.60 mm
- net N$12: track 3.12 -> 5.59 mm
- net N$13: track 5.36 -> 7.78 mm
- net N$14: track 5.75 -> 7.95 mm
- net N$16: track 6.31 -> 8.36 mm
- net N$17: track 6.86 -> 8.85 mm
- net N$6: track 2.40 -> 4.31 mm
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Other:
- board size 100 x 100 mm -> 50 x 50 mm

Commit message: final prototype
Parts:
- removed C9: (no value), rcl:C1206
- removed I2S: 1X4, headers(2mm):1X4
- removed U$4: 1X1, headers(2mm):1X1
- added C7: (no value), resistor:C0805
- added SV1: (no value), con-lstb:MA05-1
- C2: device rcl:C1206 -> resistor:C0805
- moved H4 1.14 mm to (45.0, 45.0)
- moved H2 0.58 mm to (45.0, 5.00)
- moved H1 0.36 mm to (5.00, 5.00)
- moved H3 0.32 mm to (5.00, 45.0)
Connections:
- removed net N$18: U$1.17
- net GND: now also U$1.17
- net N$12: now also C7.1; no longer C9.1
- net N$13: now also SV1.2; no longer I2S.4
- net N$14: now also SV1.3; no longer I2S.3
- net N$16: now also SV1.4; no longer I2S.2
- net N$17: now also SV1.5; no longer I2S.1
- net N$21: now also SV1.1; no longer U$4.1
- net N$5: now also C7.2; no longer C9.2
Routing:
- net N$21: track 8.60 -> 17.4 mm
- net GND: track 17.4 -> 23.6 mm
- net N$17: track 8.85 -> 12.5 mm
- net N$16: track 8.36 -> 11.7 mm
- net VCC: track 35.3 -> 38.6 mm
- net N$13: track 7.78 -> 11.1 mm
- net N$14: track 7.95 -> 10.9 mm
- net N$12: track 5.59 -> 5.00 mm
