File: boomdsp.sch (EAGLE design)
At the start: 25 parts, among them J1 RCA, J2 RCA

Commit message: proto
Parts:
- removed C1, C2: 2.2nF 50V, rcl:C-EU025-030X050
- removed GPIO: 1X4, headers(2mm):1X4
- removed J1, J2: RCA, SparkFun-Connectors:RCA
- added OUTL, OUTR: 1X2, headers(2mm):1X2
- added U$3: 1X5, headers(2mm):1X5
Connections:
- new net N$21: U$1.XSMT, U$3.5
- net GND: now also C13.2, C14.2, OUTL.1, OUTR.2; no longer C1.2, C2.2
- net N$10: now also U$3.3; no longer GPIO.3
- net N$11: now also U$3.1; no longer GPIO.1
- net N$3: now also C14.1, OUTR.1; no longer C2.1
- net N$4: now also C13.1, OUTL.2; no longer C1.1
- net N$7: now also U$3.2; no longer GPIO.2
- net N$8: now also U$3.4; no longer GPIO.4
- net VDD: no longer U$1.XSMT
Other:
- moved on the sheet: C13, C14
Changed lines of the file:
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@@
 <part name="P+1" library="supply1" deviceset="VCC" device=""/>
 <part name="P+2" library="supply1" deviceset="VCC" device=""/>
-<part name="C1" library="rcl" deviceset="C-EU" device="025-030X050" value="2.2nF 50V"/>
-<part name="C2" library="rcl" deviceset="C-EU" device="025-030X050" value="2.2nF 50V"/>
-<part name="GPIO" library="headers(2mm)" deviceset="1X4" device=""/>
 <part name="U$1" library="boomdsp" deviceset="PCM5142_I2C" device=""/>
 <part name="I2S" library="headers(2mm)" deviceset="1X4" device=""/>
@@
 <part name="GND3" library="supply1" deviceset="GND" device=""/>
 <part name="I2C" library="headers(2mm)" deviceset="1X2" device=""/>
-<part name="J1" library="SparkFun-Connectors" deviceset="RCA" device=""/>
-<part name="J2" library="SparkFun-Connectors" deviceset="RCA" device=""/>
 <part name="LED1" library="led" deviceset="LED" device="3MM"/>
 <part name="U$2" library="boomdsp" deviceset="LP5907" device=""/>
@@
 <part name="C13" library="rcl" deviceset="C-EU" device="102-043X133" value="2.2nF 50V"/>
 <part name="C14" library="rcl" deviceset="C-EU" device="102-043X133" value="2.2nF 50V"/>
+<part name="U$3" library="headers(2mm)" deviceset="1X5" device=""/>
+<part name="OUTL" library="headers(2mm)" deviceset="1X2" device=""/>
+<part name="OUTR" library="headers(2mm)" deviceset="1X2" device=""/>
+<part name="GND8" library="supply1" deviceset="GND" device=""/>
+<part name="GND9" library="supply1" deviceset="GND" device=""/>
 </parts>
 <sheets>
@@
 <instance part="P+1" gate="VCC" x="15.24" y="55.88" rot="R90"/>
 <instance part="P+2" gate="VCC" x="35.56" y="93.98"/>
-<instance part="C1" gate="G$1" x="-22.86" y="48.26"/>
-<instance part="C2" gate="G$1" x="-15.24" y="40.64"/>
-<instance part="GPIO" gate="G$1" x="71.12" y="22.86" rot="R90"/>
 <instance part="U$1" gate="G$1" x="71.12" y="58.42"/>
 <instance part="I2S" gate="G$1" x="101.6" y="58.42" rot="R180"/>
-<instance part="VDD2" gate="G$1" x="111.76" y="38.1" rot="R270"/>
+<instance part="VDD2" gate="G$1" x="111.76" y="48.26" rot="R270"/>
 <instance part="GND3" gate="1" x="111.76" y="45.72" rot="R90"/>
 <instance part="I2C" gate="G$1" x="38.1" y="35.56" rot="R90"/>
-<instance part="J1" gate="G$1" x="114.3" y="7.62"/>
-<instance part="J2" gate="G$1" x="114.3" y="-7.62"/>
 <instance part="LED1" gate="G$1" x="83.82" y="2.54"/>
 <instance part="GND5" gate="1" x="15.24" y="43.18" rot="R270"/>
@@
 <instance part="GND7" gate="1" x="30.48" y="76.2" rot="R270"/>
 <instance part="C12" gate="G$1" x="109.22" y="76.2"/>
-<instance part="C13" gate="G$1" x="-27.94" y="48.26"/>
-<instance part="C14" gate="G$1" x="-7.62" y="40.64"/>
+<instance part="C13" gate="G$1" x="-22.86" y="48.26"/>
+<instance part="C14" gate="G$1" x="-15.24" y="40.64"/>
+<instance part="U$3" gate="G$1" x="71.12" y="22.86" rot="R90"/>
+<instance part="OUTL" gate="G$1" x="-38.1" y="66.04"/>
+<instance part="OUTR" gate="G$1" x="-38.1" y="50.8"/>
+<instance part="GND8" gate="1" x="-30.48" y="48.26" rot="R90"/>
+<instance part="GND9" gate="1" x="-30.48" y="66.04" rot="R90"/>
 </instances>
 <busses>
@@
 <pinref part="R2" gate="G$1" pin="1"/>
 <wire x1="-7.62" y1="53.34" x2="-15.24" y2="53.34" width="0.1524" layer="91"/>
-<wire x1="-15.24" y1="53.34" x2="-35.56" y2="53.34" width="0.1524" layer="91"/>
-<wire x1="-15.24" y1="53.34" x2="-15.24" y2="43.18" width="0.1524" layer="91"/>
-<junction x="-15.24" y="53.34"/>
-<pinref part="C2" gate="G$1" pin="1"/>
+<wire x1="-15.24" y1="53.34" x2="-15.24" y2="50.8" width="0.1524" layer="91"/>
+<pinref part="C14" gate="G$1" pin="1"/>
+<pinref part="OUTR" gate="G$1" pin="1"/>
+<wire x1="-15.24" y1="50.8" x2="-15.24" y2="43.18" width="0.1524" layer="91"/>
+<wire x1="-15.24" y1="50.8" x2="-35.56" y2="50.8" width="0.1524" layer="91"/>
+<junction x="-15.24" y="50.8"/>
 </segment>
 </net>
@@
 <pinref part="R1" gate="G$1" pin="1"/>
 <wire x1="-7.62" y1="60.96" x2="-22.86" y2="60.96" width="0.1524" layer="91"/>
-<wire x1="-22.86" y1="60.96" x2="-35.56" y2="60.96" width="0.1524" layer="91"/>
 <wire x1="-22.86" y1="60.96" x2="-22.86" y2="50.8" width="0.1524" layer="91"/>
+<pinref part="C13" gate="G$1" pin="1"/>
+<wire x1="-22.86" y1="60.96" x2="-22.86" y2="63.5" width="0.1524" layer="91"/>
 <junction x="-22.86" y="60.96"/>
-<pinref part="C1" gate="G$1" pin="1"/>
+<pinref part="OUTL" gate="G$1" pin="2"/>
+<wire x1="-22.86" y1="63.5" x2="-35.56" y2="63.5" width="0.1524" layer="91"/>
 </segment>
 </net>
@@
 </segment>
 <segment>
-<wire x1="93.98" y1="38.1" x2="93.98" y2="48.26" width="0.1524" layer="91"/>
-<pinref part="U$1" gate="G$1" pin="XSMT"/>
-<wire x1="93.98" y1="48.26" x2="93.98" y2="66.04" width="0.1524" layer="91"/>
-<wire x1="93.98" y1="66.04" x2="86.36" y2="66.04" width="0.1524" layer="91"/>
 <pinref part="VDD2" gate="G$1" pin="VDD"/>
-<wire x1="93.98" y1="38.1" x2="109.22" y2="38.1" width="0.1524" layer="91"/>
+<wire x1="86.36" y1="48.26" x2="109.22" y2="48.26" width="0.1524" layer="91"/>
 <pinref part="U$1" gate="G$1" pin="MODE2"/>
-<wire x1="86.36" y1="48.26" x2="93.98" y2="48.26" width="0.1524" layer="91"/>
-<junction x="93.98" y="48.26"/>
 </segment>
 </net>
@@
 <wire x1="-20.32" y1="33.02" x2="-20.32" y2="30.48" width="0.1524" layer="91"/>
 <junction x="-20.32" y="33.02"/>
-<pinref part="C1" gate="G$1" pin="2"/>
-<pinref part="C2" gate="G$1" pin="2"/>
 <pinref part="GND6" gate="1" pin="GND"/>
+<pinref part="C13" gate="G$1" pin="2"/>
+<pinref part="C14" gate="G$1" pin="2"/>
 </segment>
 <segment>
@@
 <pinref part="GND7" gate="1" pin="GND"/>
 </segment>
+<segment>
+<pinref part="GND9" gate="1" pin="GND"/>
+<pinref part="OUTL" gate="G$1" pin="1"/>
+<wire x1="-33.02" y1="66.04" x2="-35.56" y2="66.04" width="0.1524" layer="91"/>
+</segment>
+<segment>
+<pinref part="GND8" gate="1" pin="GND"/>
+<pinref part="OUTR" gate="G$1" pin="2"/>
+<wire x1="-33.02" y1="48.26" x2="-35.56" y2="48.26" width="0.1524" layer="91"/>
+</segment>
 </net>
 <net name="VCC" class="0">
@@
 <wire x1="88.9" y1="30.48" x2="68.58" y2="30.48" width="0.1524" layer="91"/>
 <pinref part="U$1" gate="G$1" pin="GPIO3"/>
-<pinref part="GPIO" gate="G$1" pin="2"/>
 <wire x1="68.58" y1="30.48" x2="68.58" y2="25.4" width="0.1524" layer="91"/>
+<pinref part="U$3" gate="G$1" pin="2"/>
 </segment>
 </net>
@@
 <wire x1="55.88" y1="40.64" x2="53.34" y2="40.64" width="0.1524" layer="91"/>
 <wire x1="53.34" y1="40.64" x2="53.34" y2="27.94" width="0.1524" layer="91"/>
-<pinref part="GPIO" gate="G$1" pin="4"/>
 <wire x1="53.34" y1="27.94" x2="73.66" y2="27.94" width="0.1524" layer="91"/>
 <wire x1="73.66" y1="27.94" x2="73.66" y2="25.4" width="0.1524" layer="91"/>
 <pinref part="U$1" gate="G$1" pin="GPIO4"/>
+<pinref part="U$3" gate="G$1" pin="4"/>
 </segment>
 </net>
@@
 <wire x1="50.8" y1="43.18" x2="50.8" y2="35.56" width="0.1524" layer="91"/>
 <wire x1="50.8" y1="35.56" x2="71.12" y2="35.56" width="0.1524" layer="91"/>
-<pinref part="GPIO" gate="G$1" pin="3"/>
 <wire x1="71.12" y1="35.56" x2="71.12" y2="25.4" width="0.1524" layer="91"/>
 <pinref part="U$1" gate="G$1" pin="GPIO5"/>
+<pinref part="U$3" gate="G$1" pin="3"/>
 </segment>
 </net>
@@
 <wire x1="91.44" y1="33.02" x2="66.04" y2="33.02" width="0.1524" layer="91"/>
 <pinref part="U$1" gate="G$1" pin="GPIO6"/>
-<pinref part="GPIO" gate="G$1" pin="1"/>
 <wire x1="66.04" y1="33.02" x2="66.04" y2="25.4" width="0.1524" layer="91"/>
+<pinref part="U$3" gate="G$1" pin="1"/>
 </segment>
 </net>
@@
 </segment>
 </net>
+<net name="N$21" class="0">
+<segment>
+<pinref part="U$1" gate="G$1" pin="XSMT"/>
+<wire x1="86.36" y1="66.04" x2="93.98" y2="66.04" width="0.1524" layer="91"/>
+<wire x1="93.98" y1="66.04" x2="93.98" y2="27.94" width="0.1524" layer="91"/>
+<pinref part="U$3" gate="G$1" pin="5"/>
+<wire x1="93.98" y1="27.94" x2="76.2" y2="27.94" width="0.1524" layer="91"/>
+<wire x1="76.2" y1="27.94" x2="76.2" y2="25.4" width="0.1524" layer="91"/>
+</segment>
+</net>

Commit message: finished prototype
Parts:
- removed C10, C11: 1uF, rcl:C-EUC0805
- removed C12: (no value), rcl:C-EUC0603K
- removed C9: 10uF 16V, rcl:CPOL-EU153CLV-0405
- removed LED1: (no value), led:LED3MM
- removed U$3: 1X5, headers(2mm):1X5
- added C1: (no value), rcl:CPOL-EUE3.5-8
- added POWER1: 1X2, headers(2mm):1X2
- added U$4: 1X1, headers(2mm):1X1
- U$2: value LP5907 -> 1X4; device boomdsp:LP5907 -> headers(2mm):1X4
Connections:
- removed net +5V: C10.1, POWER.1, U$2.EN, U$2.IN
- removed net VDD: C4.1, U$1.DVDD, U$1.MODE2
- net GND: now also C1.-, POWER1.2, U$1.ADR1, U$1.ADR2; no longer C10.2, C11.2, C9.-, U$2.GND
- net N$10: now also U$2.3; no longer U$3.3
- net N$11: now also U$2.1; no longer U$3.1
- net N$15: now also C1.+; no longer C9.+
- net N$21: now also U$4.1; no longer U$3.5
- net N$7: now also U$2.2; no longer U$3.2
- net N$8: now also U$2.4; no longer U$3.4
- net VCC: now also C4.1, POWER.1, POWER1.1, U$1.DVDD, U$1.MODE2; no longer C11.1, U$2.OUT

Commit message: damn vias
Parts:
- removed C5, C7: 2.2uF 25V, rcl:C-EUC0805
- removed I2C: 1X2, headers(2mm):1X2
- removed U$2: 1X4, headers(2mm):1X4
- added C2, C9: (no value), rcl:C-EUC1206
- added H1, H2, H3, H4: MOUNT-HOLE3.2, holes:MOUNT-HOLE3.2
- added SV2: (no value), con-lstb:MA06-1
Connections:
- net GND: now also C2.1; no longer C5.1
- net N$10: now also SV2.4; no longer U$2.3
- net N$11: now also SV2.6; no longer U$2.1
- net N$12: now also C9.1; no longer C7.1
- net N$19: now also SV2.1; no longer I2C.1
- net N$20: now also SV2.2; no longer I2C.2
- net N$5: now also C9.2; no longer C7.2
- net N$7: now also SV2.5; no longer U$2.2
- net N$8: now also SV2.3; no longer U$2.4
- net N$9: now also C2.2; no longer C5.2
Changed lines of the file:
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@@
 <part name="C3" library="rcl" deviceset="C-EU" device="C0805" value="0.1uF 100V"/>
 <part name="C4" library="rcl" deviceset="C-EU" device="C0805" value="0.1uF 100V"/>
-<part name="C5" library="rcl" deviceset="C-EU" device="C0805" value="2.2uF 25V"/>
 <part name="C6" library="rcl" deviceset="C-EU" device="C0805" value="0.1uF 100V"/>
-<part name="C7" library="rcl" deviceset="C-EU" device="C0805" value="2.2uF 25V"/>
 <part name="C8" library="rcl" deviceset="C-EU" device="C0805" value="0.1uF 100V"/>
 <part name="GND1" library="supply1" deviceset="GND" device=""/>
@@
 <part name="I2S" library="headers(2mm)" deviceset="1X4" device=""/>
 <part name="GND3" library="supply1" deviceset="GND" device=""/>
-<part name="I2C" library="headers(2mm)" deviceset="1X2" device=""/>
 <part name="POWER" library="headers(2mm)" deviceset="1X2" device=""/>
 <part name="GND2" library="supply1" deviceset="GND" device=""/>
@@
 <part name="GND11" library="supply1" deviceset="GND" device=""/>
 <part name="C1" library="rcl" deviceset="CPOL-EU" device="E3.5-8"/>
-<part name="U$2" library="headers(2mm)" deviceset="1X4" device=""/>
 <part name="U$4" library="headers(2mm)" deviceset="1X1" device=""/>
 <part name="P+5" library="supply1" deviceset="VCC" device=""/>
 <part name="P+6" library="supply1" deviceset="VCC" device=""/>
+<part name="SV2" library="con-lstb" deviceset="MA06-1" device=""/>
+<part name="H1" library="holes" deviceset="MOUNT-HOLE" device="3.2"/>
+<part name="H2" library="holes" deviceset="MOUNT-HOLE" device="3.2"/>
+<part name="H3" library="holes" deviceset="MOUNT-HOLE" device="3.2"/>
+<part name="H4" library="holes" deviceset="MOUNT-HOLE" device="3.2"/>
+<part name="C9" library="rcl" deviceset="C-EU" device="C1206"/>
+<part name="C2" library="rcl" deviceset="C-EU" device="C1206"/>
 </parts>
 <sheets>
@@
 <instance part="C3" gate="G$1" x="101.6" y="76.2"/>
 <instance part="C4" gate="G$1" x="101.6" y="88.9"/>
-<instance part="C5" gate="G$1" x="35.56" y="71.12"/>
 <instance part="C6" gate="G$1" x="35.56" y="83.82"/>
-<instance part="C7" gate="G$1" x="15.24" y="73.66"/>
 <instance part="C8" gate="G$1" x="20.32" y="50.8"/>
 <instance part="GND1" gate="1" x="119.38" y="81.28" rot="R90"/>
@@
 <instance part="I2S" gate="G$1" x="101.6" y="58.42" rot="R180"/>
 <instance part="GND3" gate="1" x="111.76" y="45.72" rot="R90"/>
-<instance part="I2C" gate="G$1" x="38.1" y="35.56" rot="R90"/>
 <instance part="GND5" gate="1" x="15.24" y="43.18" rot="R270"/>
 <instance part="GND6" gate="1" x="-20.32" y="27.94"/>
@@
 <instance part="GND11" gate="1" x="111.76" y="63.5" rot="R90"/>
 <instance part="C1" gate="G$1" x="20.32" y="35.56" rot="R180"/>
-<instance part="U$2" gate="G$1" x="71.12" y="22.86" rot="R90"/>
 <instance part="U$4" gate="G$1" x="93.98" y="22.86" rot="R90"/>
+<instance part="SV2" gate="1" x="71.12" y="12.7" rot="R90"/>
+<instance part="C9" gate="G$1" x="15.24" y="73.66"/>
+<instance part="C2" gate="G$1" x="35.56" y="71.12"/>
 </instances>
 <busses>
@@
 <net name="N$9" class="0">
 <segment>
-<pinref part="C5" gate="G$1" pin="2"/>
 <wire x1="55.88" y1="63.5" x2="35.56" y2="63.5" width="0.1524" layer="91"/>
 <wire x1="35.56" y1="63.5" x2="35.56" y2="66.04" width="0.1524" layer="91"/>
 <pinref part="U$1" gate="G$1" pin="VNEG"/>
+<pinref part="C2" gate="G$1" pin="2"/>
 </segment>
 </net>
 <net name="N$5" class="0">
 <segment>
-<pinref part="C7" gate="G$1" pin="2"/>
 <wire x1="55.88" y1="66.04" x2="15.24" y2="66.04" width="0.1524" layer="91"/>
 <wire x1="15.24" y1="66.04" x2="15.24" y2="68.58" width="0.1524" layer="91"/>
 <pinref part="U$1" gate="G$1" pin="CAPM"/>
+<pinref part="C9" gate="G$1" pin="2"/>
 </segment>
 </net>
@@
 <wire x1="55.88" y1="71.12" x2="45.72" y2="71.12" width="0.1524" layer="91"/>
 <wire x1="45.72" y1="71.12" x2="45.72" y2="78.74" width="0.1524" layer="91"/>
-<pinref part="C7" gate="G$1" pin="1"/>
 <wire x1="45.72" y1="78.74" x2="15.24" y2="78.74" width="0.1524" layer="91"/>
 <wire x1="15.24" y1="78.74" x2="15.24" y2="76.2" width="0.1524" layer="91"/>
 <pinref part="U$1" gate="G$1" pin="CAPP"/>
+<pinref part="C9" gate="G$1" pin="1"/>
 </segment>
 </net>
@@
 <wire x1="55.88" y1="68.58" x2="43.18" y2="68.58" width="0.1524" layer="91"/>
 <wire x1="43.18" y1="68.58" x2="43.18" y2="76.2" width="0.1524" layer="91"/>
-<pinref part="C5" gate="G$1" pin="1"/>
 <wire x1="43.18" y1="76.2" x2="35.56" y2="76.2" width="0.1524" layer="91"/>
 <wire x1="35.56" y1="76.2" x2="35.56" y2="73.66" width="0.1524" layer="91"/>
@@
 <pinref part="U$1" gate="G$1" pin="CPGND"/>
 <pinref part="GND7" gate="1" pin="GND"/>
+<pinref part="C2" gate="G$1" pin="1"/>
 </segment>
 <segment>
@@
 <wire x1="88.9" y1="30.48" x2="68.58" y2="30.48" width="0.1524" layer="91"/>
 <pinref part="U$1" gate="G$1" pin="GPIO3"/>
-<wire x1="68.58" y1="30.48" x2="68.58" y2="25.4" width="0.1524" layer="91"/>
-<pinref part="U$2" gate="G$1" pin="2"/>
+<pinref part="SV2" gate="1" pin="5"/>
+<wire x1="68.58" y1="30.48" x2="68.58" y2="20.32" width="0.1524" layer="91"/>
 </segment>
 </net>
@@
 <wire x1="53.34" y1="40.64" x2="53.34" y2="27.94" width="0.1524" layer="91"/>
 <wire x1="53.34" y1="27.94" x2="73.66" y2="27.94" width="0.1524" layer="91"/>
-<wire x1="73.66" y1="27.94" x2="73.66" y2="25.4" width="0.1524" layer="91"/>
 <pinref part="U$1" gate="G$1" pin="GPIO4"/>
-<pinref part="U$2" gate="G$1" pin="4"/>
+<pinref part="SV2" gate="1" pin="3"/>
+<wire x1="73.66" y1="27.94" x2="73.66" y2="20.32" width="0.1524" layer="91"/>
 </segment>
 </net>
@@
 <wire x1="50.8" y1="43.18" x2="50.8" y2="35.56" width="0.1524" layer="91"/>
 <wire x1="50.8" y1="35.56" x2="71.12" y2="35.56" width="0.1524" layer="91"/>
-<wire x1="71.12" y1="35.56" x2="71.12" y2="25.4" width="0.1524" layer="91"/>
+<wire x1="71.12" y1="35.56" x2="71.12" y2="20.32" width="0.1524" layer="91"/>
 <pinref part="U$1" gate="G$1" pin="GPIO5"/>
-<pinref part="U$2" gate="G$1" pin="3"/>
+<pinref part="SV2" gate="1" pin="4"/>
 </segment>
 </net>
@@
 <wire x1="91.44" y1="33.02" x2="66.04" y2="33.02" width="0.1524" layer="91"/>
 <pinref part="U$1" gate="G$1" pin="GPIO6"/>
-<wire x1="66.04" y1="33.02" x2="66.04" y2="25.4" width="0.1524" layer="91"/>
-<pinref part="U$2" gate="G$1" pin="1"/>
+<wire x1="66.04" y1="33.02" x2="66.04" y2="20.32" width="0.1524" layer="91"/>
+<pinref part="SV2" gate="1" pin="6"/>
 </segment>
 </net>
@@
 <segment>
 <pinref part="U$1" gate="G$1" pin="SDA"/>
-<pinref part="I2C" gate="G$1" pin="1"/>
 <wire x1="55.88" y1="48.26" x2="38.1" y2="48.26" width="0.1524" layer="91"/>
-<wire x1="38.1" y1="48.26" x2="38.1" y2="38.1" width="0.1524" layer="91"/>
+<wire x1="38.1" y1="48.26" x2="38.1" y2="22.86" width="0.1524" layer="91"/>
+<wire x1="38.1" y1="22.86" x2="78.74" y2="22.86" width="0.1524" layer="91"/>
+<pinref part="SV2" gate="1" pin="1"/>
+<wire x1="78.74" y1="22.86" x2="78.74" y2="20.32" width="0.1524" layer="91"/>
 </segment>
 </net>
@@
 <segment>
 <pinref part="U$1" gate="G$1" pin="SCL"/>
-<pinref part="I2C" gate="G$1" pin="2"/>
 <wire x1="55.88" y1="45.72" x2="40.64" y2="45.72" width="0.1524" layer="91"/>
-<wire x1="40.64" y1="45.72" x2="40.64" y2="38.1" width="0.1524" layer="91"/>
+<wire x1="40.64" y1="45.72" x2="40.64" y2="25.4" width="0.1524" layer="91"/>
+<wire x1="40.64" y1="25.4" x2="76.2" y2="25.4" width="0.1524" layer="91"/>
+<pinref part="SV2" gate="1" pin="2"/>
+<wire x1="76.2" y1="25.4" x2="76.2" y2="20.32" width="0.1524" layer="91"/>
 </segment>
 </net>
@@
 <instance part="P+5" gate="VCC" x="30.48" y="86.36" rot="R270"/>
 <instance part="P+6" gate="VCC" x="30.48" y="71.12" rot="R270"/>
+<instance part="H1" gate="G$1" x="55.88" y="83.82"/>
+<instance part="H2" gate="G$1" x="55.88" y="76.2"/>
+<instance part="H3" gate="G$1" x="55.88" y="68.58"/>
+<instance part="H4" gate="G$1" x="55.88" y="60.96"/>
 </instances>
 <busses>
